File: LED-Stack/LED/LED.kicad_pcb (KiCad board)
At the start: 2 copper layers, 15.6 x 9.8 mm, 10 parts, among them J1 VCC, J2 Conn_01x01, J3 Conn_01x01, J4 GND, SW1 SW_SPST

Commit message: Update LED stack 3D renderings.
Parts:
- LED Symbol: renamed from Ref**
Changed lines of the file:
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@@
       (padsonsilk false)
       (subtractmaskfromsilk false)
-      (outputformat 1)
+      (outputformat 5)
       (mirror false)
-      (drillshape 1)
+      (drillshape 0)
       (scaleselection 1)
-      (outputdirectory ""))
+      (outputdirectory "./rendering/layers/"))
   )
   (net 0 "")
@@
     (add_net "Net-(J2-Pad1)")
     (add_net "Net-(J3-Pad1)")
+  )
+  (module project-lib:LED_symbol (layer B.Cu)
+    (at 100.02 96.94)
+    (fp_text reference "LED Symbol" (at 0 0) (layer B.SilkS) hide
+      (effects (font (size 1.27 1.27) (thickness 0.15)) (justify mirror))
+    )
+    (fp_text value Val** (at 0 0) (layer B.SilkS) hide
+      (effects (font (size 1.27 1.27) (thickness 0.15)) (justify mirror))
+    )
+    (fp_line (start 0.39 0.67) (end 0.2 0.6) (layer B.SilkS) (width 0.12))
+    (fp_line (start 0.39 0.67) (end 0.42 0.47) (layer B.SilkS) (width 0.12))
+    (fp_line (start 0.18 0.32) (end 0.39 0.67) (layer B.SilkS) (width 0.12))
+    (fp_line (start -0.01 0.87) (end 0.02 0.67) (layer B.SilkS) (width 0.12))
+    (fp_line (start -0.01 0.87) (end -0.2 0.8) (layer B.SilkS) (width 0.12))
+    (fp_line (start -0.22 0.52) (end -0.01 0.87) (layer B.SilkS) (width 0.12))
+    (fp_line (start -1.97 -0.25) (end -0.42 -0.25) (layer B.SilkS) (width 0.12))
+    (fp_line (start -0.42 -0.25) (end -0.42 0.26) (layer B.SilkS) (width 0.12))
+    (fp_line (start -0.42 -0.27) (end -0.42 -0.78) (layer B.SilkS) (width 0.12))
+    (fp_line (start 0.44 -0.26) (end 0.44 0.25) (layer B.SilkS) (width 0.12))
+    (fp_line (start 0.44 -0.26) (end 0.44 -0.77) (layer B.SilkS) (width 0.12))
+    (fp_line (start 0.44 -0.26) (end -0.42 0.26) (layer B.SilkS) (width 0.12))
+    (fp_line (start 0.44 -0.26) (end -0.42 -0.78) (layer B.SilkS) (width 0.12))
+    (fp_line (start 1.95 -0.25) (end 0.44 -0.25) (layer B.SilkS) (width 0.12))
   )
   (module project-lib:Connection_Points (layer F.Cu)
@@
       (xy 0.042145 0.989873)) (layer B.SilkS) (width 0.01))
   )
-  (module project-lib:LED_symbol (layer B.Cu)
-    (at 100.02 96.94)
-    (fp_text reference Ref** (at 0 0) (layer B.SilkS) hide
-      (effects (font (size 1.27 1.27) (thickness 0.15)) (justify mirror))
-    )
-    (fp_text value Val** (at 0 0) (layer B.SilkS) hide
-      (effects (font (size 1.27 1.27) (thickness 0.15)) (justify mirror))
-    )
-    (fp_poly (pts (xy 0.176385 0.774361) (xy 0.207452 0.728215) (xy 0.224209 0.663752) (xy 0.225984 0.59822)
-      (xy 0.201248 0.564898) (xy 0.151015 0.564622) (xy 0.127017 0.55804) (xy 0.097369 0.523398)
-      (xy 0.058456 0.455909) (xy 0.037115 0.413861) (xy -0.015103 0.31962) (xy -0.058233 0.266499)
-      (xy -0.092497 0.254323) (xy -0.118117 0.282915) (xy -0.120384 0.288456) (xy -0.117684 0.323881)
-      (xy -0.097502 0.386064) (xy -0.063222 0.464931) (xy -0.056219 0.479306) (xy -0.015581 0.561901)
-      (xy 0.00822 0.613698) (xy 0.017038 0.641881) (xy 0.012727 0.653634) (xy -0.00286 0.656143)
-      (xy -0.010583 0.656167) (xy -0.036718 0.673672) (xy -0.042333 0.69651) (xy -0.027442 0.728927)
-      (xy 0.021224 0.757465) (xy 0.052747 0.769251) (xy 0.127249 0.786544) (xy 0.176385 0.774361)) (layer B.SilkS) (width 0.01))
-    (fp_poly (pts (xy 0.474884 0.642962) (xy 0.503045 0.597429) (xy 0.50593 0.589508) (xy 0.527 0.504843)
-      (xy 0.521257 0.449927) (xy 0.506156 0.432777) (xy 0.473234 0.432812) (xy 0.459493 0.442207)
-      (xy 0.441764 0.443447) (xy 0.415748 0.415439) (xy 0.378452 0.35434) (xy 0.350212 0.301721)
-      (xy 0.294791 0.20648) (xy 0.247516 0.147867) (xy 0.209762 0.127056) (xy 0.182904 0.145223)
-      (xy 0.178452 0.154934) (xy 0.181917 0.187327) (xy 0.201701 0.245783) (xy 0.233862 0.319191)
-      (xy 0.244263 0.340347) (xy 0.282009 0.417144) (xy 0.301918 0.465477) (xy 0.306012 0.494268)
-      (xy 0.296315 0.512438) (xy 0.285342 0.521499) (xy 0.260983 0.556668) (xy 0.271569 0.593732)
-      (xy 0.310464 0.626649) (xy 0.371031 0.649374) (xy 0.433224 0.656167) (xy 0.474884 0.642962)) (layer B.SilkS) (width 0.01))
-    (fp_poly (pts (xy -0.400066 0.306947) (xy -0.341336 0.27752) (xy -0.258352 0.232439) (xy -0.15703 0.174945)
-      (xy -0.043285 0.108278) (xy -0.005994 0.085995) (xy 0.379595 -0.145471) (xy 0.385589 0.080723)
-      (xy 0.388717 0.180889) (xy 0.392915 0.246417) (xy 0.399955 0.284998) (xy 0.411607 0.304319)
-      (xy 0.42964 0.312072) (xy 0.439209 0.313681) (xy 0.459233 0.315127) (xy 0.472672 0.308154)
-      (xy 0.480839 0.285913) (xy 0.485046 0.241556) (xy 0.486607 0.168234) (xy 0.486834 0.065243)
-      (xy 0.486834 -0.189958) (xy 1.232959 -0.195521) (xy 1.979084 -0.201083) (xy 1.985847 -0.248708)
-      (xy 1.992611 -0.296333) (xy 0.486834 -0.296333) (xy 0.486834 -0.549084) (xy 0.485151 -0.67022)
-      (xy 0.479308 -0.753167) (xy 0.468113 -0.801967) (xy 0.450377 -0.820661) (xy 0.424907 -0.81329)
-      (xy 0.411823 -0.803564) (xy 0.396451 -0.778744) (xy 0.386804 -0.730498) (xy 0.381985 -0.652001)
-      (xy 0.381 -0.568908) (xy 0.380127 -0.480646) (xy 0.377776 -0.410808) (xy 0.374346 -0.368408)
-      (xy 0.37172 -0.359833) (xy 0.351606 -0.370244) (xy 0.300822 -0.399302) (xy 0.224925 -0.44375)
-      (xy 0.12947 -0.500329) (xy 0.020013 -0.565779) (xy -0.006371 -0.581631) (xy -0.140739 -0.662289)
-      (xy -0.243474 -0.723373) (xy -0.319145 -0.767252) (xy -0.372322 -0.796293) (xy -0.407575 -0.812865)
-      (xy -0.429473 -0.819337) (xy -0.442585 -0.818078) (xy -0.450897 -0.812047) (xy -0.456671 -0.786228)
-      (xy -0.461387 -0.726976) (xy -0.46455 -0.643188) (xy -0.465666 -0.546805) (xy -0.465666 -0.296333)
-      (xy -1.971444 -0.296333) (xy -1.964251 -0.245684) (xy -0.359833 -0.245684) (xy -0.359064 -0.371991)
-      (xy -0.35692 -0.481819) (xy -0.353646 -0.568933) (xy -0.349487 -0.627091) (xy -0.344688 -0.650055)
-      (xy -0.343958 -0.650096) (xy -0.321212 -0.6369) (xy -0.268535 -0.605931) (xy -0.192407 -0.561011)
-      (xy -0.09931 -0.505961) (xy -0.03175 -0.465954) (xy 0.070266 -0.404978) (xy 0.160608 -0.349978)
-      (xy 0.232431 -0.305198) (xy 0.278892 -0.274885) (xy 0.292073 -0.265112) (xy 0.295082 -0.251826)
-      (xy 0.278949 -0.230988) (xy 0.239945 -0.199866) (xy 0.174342 -0.155727) (xy 0.07841 -0.095838)
-      (xy -0.020136 -0.036273) (xy -0.359833 0.167296) (xy -0.359833 -0.245684) (xy -1.964251 -0.245684)
-      (xy -1.957916 -0.201083) (xy -1.211791 -0.195521) (xy -0.465666 -0.189958) (xy -0.465666 0.063771)
-      (xy -0.465097 0.171526) (xy -0.462718 0.243846) (xy -0.457523 0.287624) (xy -0.448506 0.309749)
-      (xy -0.434661 0.317114) (xy -0.428625 0.31748) (xy -0.400066 0.306947)) (layer B.SilkS) (width 0.01))
-  )
   (module Connector_PinHeader_2.54mm:PinHeader_1x01_P2.54mm_Vertical (layer F.Cu)
     (at 106.33 96.19)
@@
   )
   (gr_line (start 95.32 95.96) (end 104.72 95.94) (layer Edge.Cuts) (width 0.05))
-  (gr_line (start 98.17 96.69) (end 94.43 96.69) (layer B.SilkS) (width 0.11))
-  (gr_line (start 101.82 96.69) (end 105.52 96.69) (layer B.SilkS) (width 0.11))
+  (gr_line (start 98.17 96.69) (end 94.43 96.69) (layer B.SilkS) (width 0.12))
+  (gr_line (start 101.82 96.69) (end 105.52 96.69) (layer B.SilkS) (width 0.12))
   (gr_arc (start 92.980016 95.889999) (end 92.975017 95.14) (angle -89.6180338) (layer Edge.Cuts) (width 0.05))
   (gr_arc (start 107.029999 95.874999) (end 107.779998 95.87) (angle -89.6180338) (layer Edge.Cuts) (width 0.05))
